File: schematics/cubeSchem/blinky-power-mon-cube.kicad_pcb (KiCad board)
At the start: 2 copper layers, 125 x 78 mm, 18 parts, among them J1 VACout, J2 VACin, J3 CTin, J4 CTout, J5 4-20mA, J6 TripStatus, J7 SMA Ant, U2 ACS712_20, U3 FEATHER_M0_BASIC_PROTO

Commit message: added logo
Parts:
- added G***: LOGO, dmcginnis427Footprints:blmcLogo2, F.Cu at (216.0, 87.0)

Commit message: updating power-mon-schem
Parts:
- removed D3.3V1: D_Zener, Diode_THT:D_DO-35_SOD27_P7.62mm_Horizontal
- removed G***: LOGO, dmcginnis427Footprints:blmcLogo2
- removed R2: 1k, Resistor_THT:R_Axial_DIN0207_L6.3mm_D2.5mm_P10.16mm_Horizontal
- added C1: 0.1uF, Capacitor_SMD:C_1206_3216Metric_Pad1.42x1.75mm_HandSolder, B.Cu at (202.5, 89.5)
- added C2: 1uF, Capacitor_SMD:C_1206_3216Metric_Pad1.42x1.75mm_HandSolder, B.Cu at (107.5, 116.5)
- added C3: 0.1uF, Capacitor_SMD:C_1206_3216Metric_Pad1.42x1.75mm_HandSolder, B.Cu at (184.5, 111.5)
- added C5: 0.1uF, Capacitor_SMD:C_1206_3216Metric_Pad1.42x1.75mm_HandSolder, B.Cu at (203.5, 96.0)
- added REF**: Lipo1500, dmcginnis427Footprints:Lipo1500, F.Cu at (150.5, 105.5)
- added U4: AMAX31865, dmcginnis427Footprints:AMAX31865, F.Cu at (202.0, 100.0)
- J5: value 4-20mA -> Reed
- R1: value 100 -> 10k; footprint Resistor_THT:R_Axial_DIN0207_L6.3mm_D2.5mm_P10.16mm_Horizontal -> Resistor_SMD:R_1206_3216Metric_Pad1.42x1.75mm_HandSolder; moved to B.Cu
- R3, R4, R5, R6: footprint Resistor_THT:R_Axial_DIN0207_L6.3mm_D2.5mm_P10.16mm_Horizontal -> Resistor_SMD:R_1206_3216Metric_Pad1.42x1.75mm_HandSolder; moved to B.Cu
- U2: footprint dmcginnis427:ACS712_20A -> dmcginnis427Footprints:ACS712_20A
- moved TP1 91.0 mm to (212.7, 123.2)
- moved J7 88.3 mm to (217.0, 113.0)
- moved R1 71.1 mm to (171.0, 66.5), turned to 90 degrees
- moved J5 60.1 mm to (176.1, 75.0), turned to 180 degrees
- moved PS1 57.9 mm to (114.4, 90.8), turned to 270 degrees
- moved U3 53.9 mm to (188.4, 116.8), turned to 0 degrees
- moved J2 49.7 mm to (143.5, 71.0), turned to 180 degrees
- moved J1 36.7 mm to (133.5, 110.0), turned to 0 degrees
- moved J6 28.8 mm to (193.0, 75.0), turned to 180 degrees
- moved R4 22.2 mm to (193.0, 66.5), turned to 90 degrees
- moved R3 20.3 mm to (183.0, 66.5), turned to 270 degrees
- moved J4 16.7 mm to (156.5, 94.0)
- moved R6 16.5 mm to (181.0, 88.0), turned to 270 degrees
- moved J3 15.3 mm to (156.5, 85.0)
- moved U2 9.12 mm to (195.0, 89.5)
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Connections:
- J1 pad 3: GND -> Net-(J1-Pad3)
- J2 pad 1: GND -> Net-(J2-Pad1)
- J2 pad 2: Net-(J2-Pad2) -> Net-(J1-Pad2)
- J3 pad 1: Net-(J2-Pad2) -> Net-(J2-Pad1)
- J4 pad 1: Net-(J1-Pad2) -> Net-(J1-Pad3)
- J5 pad 1: Net-(J5-Pad1) -> +3V3
- J5 pad 2: GND -> Net-(J5-Pad2)
- J6 pad 2: Net-(J6-Pad2) -> +3V3
- PS1 pad 1: Net-(J2-Pad2) -> Net-(J2-Pad1)
- R1 pad 1: Net-(J5-Pad1) -> Net-(J5-Pad2)
- U3 pad P1_15: Net-(J6-Pad2) -> +3V3
- U3 pad P1_9: Net-(U3-PadP1_9) -> Net-(J5-Pad2)
- U3 pad P2_10: Net-(U3-PadP2_10) -> Net-(J6-Pad1)
- U3 pad P2_5: Net-(J6-Pad3) -> Net-(U3-PadP2_5)
- U3 pad P2_6: Net-(J6-Pad1) -> Net-(U3-PadP2_6)
- U3 pad P2_9: Net-(U3-PadP2_9) -> Net-(J6-Pad3)
Routing:
- net Net-(J1-Pad1): track 92.6 -> 0.00 mm
- net Net-(J6-Pad3): track 76.4 -> 0.00 mm
- net Net-(U3-PadP1_14): track 73.8 -> 0.00 mm
- net Net-(J6-Pad1): track 66.8 -> 0.00 mm, vias 1 -> 0
- net +5V: track 50.1 -> 0.00 mm
- net Net-(J2-Pad2): track 48.5 -> 0.00 mm
- net Net-(J1-Pad2): track 39.0 -> 0.00 mm
- net Net-(J6-Pad2): track 37.1 -> 0.00 mm
- net Net-(R5-Pad1): track 36.7 -> 0.00 mm
- net Net-(J5-Pad1): track 15.9 -> 0.00 mm
- net Net-(J7-Pad1): track 11.4 -> 0.00 mm
- net Net-(R5-Pad2): track 8.67 -> 0.00 mm
- net GND: vias 10 -> 0
- removed copper zone on B.Cu, net GND
- removed copper zone on F.Cu, net GND
Other:
- outline, holes or cut-outs redrawn
- board text removed: "Blinky-Power-Mon-V1.0"

Commit message: laying out pcb for temp mon
Parts:
- moved R5 0.51 mm to (187.0, 89.5), turned to 0 degrees
- moved J1 0.16 mm to (133.3, 110.0)
Routing:
- net +3V3: track 0.00 -> 121.5 mm
- net +5V: track 0.00 -> 105.7 mm, vias 0 -> 1
- net Net-(J5-Pad2): track 0.00 -> 65.7 mm, vias 0 -> 1
- net Net-(J6-Pad3): track 0.00 -> 51.3 mm
- net Net-(R5-Pad1): track 0.00 -> 45.6 mm
- net Net-(J6-Pad1): track 0.00 -> 43.6 mm
- net Net-(J1-Pad1): track 0.00 -> 30.6 mm
- net Net-(U3-PadP2_5): track 0.00 -> 27.2 mm
- net Net-(U3-PadP2_4): track 0.00 -> 27.2 mm
- net Net-(U3-PadP2_7): track 0.00 -> 27.0 mm
- net Net-(U3-PadP2_6): track 0.00 -> 27.0 mm
- net Net-(J2-Pad1): track 0.00 -> 21.0 mm
- net Net-(J7-Pad1): track 0.00 -> 12.4 mm
- net Net-(R5-Pad2): track 0.00 -> 6.52 mm

Commit message: pcb design seems finished
Parts:
- removed REF**: Lipo1500, dmcginnis427Footprints:Lipo1500
- added ACG1: TestPoint, TestPoint:TestPoint_THTPad_3.0x3.0mm_Drill1.5mm, F.Cu at (150.0, 110.0)
- added DCG1: TestPoint, TestPoint:TestPoint_THTPad_3.0x3.0mm_Drill1.5mm, F.Cu at (160.0, 110.0)
- added G***: LOGO, dmcginnis427Footprints:blmcLogo2_bs, F.Cu at (118.0, 90.5)
- added G***: LOGO, dmcginnis427Footprints:blmcLogo, F.Cu at (175.0, 58.0)
- added Lipo1500bs: Lipo1500_bs, dmcginnis427Footprints:Lipo1500_bs, F.Cu at (100.5, 105.5)
- added Lipo1500fs: Lipo1500, dmcginnis427Footprints:Lipo1500, F.Cu at (100.5, 75.5)
Routing:
- net Net-(ACG1-Pad1): track 0.00 -> 59.3 mm
- net Net-(J1-Pad1): track 30.6 -> 69.6 mm
- net Net-(J1-Pad3): track 0.00 -> 25.6 mm
- net Net-(J2-Pad1): track 21.0 -> 43.6 mm
- net +5V: track 105.7 -> 124.7 mm
- net +3V3: track 121.5 -> 124.8 mm
- net GND: vias 0 -> 14
- added copper zone on B.Cu, net GND
- added copper zone on F.Cu, net GND
Other:
- board text added: "Blinky Fridge Monitor v1.0"
