File: schematics/cubeSchem/blinky-power-mon-cube.sch (KiCad schematic (older format))
At the start: 18 parts, among them J1 VACout, J2 VACin, J3 CTin, J4 CTout, J5 4-20mA, J6 TripStatus, J7 SMA Ant, U2 ACS712_20, U3 FEATHER_M0_BASIC_PROTO

Commit message: updating power-mon-schem
Parts:
- removed D3.3V1: D_Zener, Diode_THT:D_DO-35_SOD27_P7.62mm_Horizontal, symbol Device:D_Zener
- removed R2: 1k, Resistor_THT:R_Axial_DIN0207_L6.3mm_D2.5mm_P10.16mm_Horizontal, symbol Device:R
- added C1, C3, C5: 0.1uF, Capacitor_SMD:C_1206_3216Metric_Pad1.42x1.75mm_HandSolder, symbol Device:C
- added C2: 1uF, Capacitor_SMD:C_1206_3216Metric_Pad1.42x1.75mm_HandSolder, symbol Device:C
- added U4: AMAX31865, dmcginnis427Footprints:AMAX31865, symbol dmcginnis427:AMAX31865
- J5: value 4-20mA -> Reed
- R1: value 100 -> 10k; footprint Resistor_THT:R_Axial_DIN0207_L6.3mm_D2.5mm_P10.16mm_Horizontal -> Resistor_SMD:R_1206_3216Metric_Pad1.42x1.75mm_HandSolder
- R3, R4, R5, R6: footprint Resistor_THT:R_Axial_DIN0207_L6.3mm_D2.5mm_P10.16mm_Horizontal -> Resistor_SMD:R_1206_3216Metric_Pad1.42x1.75mm_HandSolder
- U2: footprint dmcginnis427:ACS712_20A -> dmcginnis427Footprints:ACS712_20A
Connections:
- net +5V: now also C1.2, C2.1, C3.2
- net GND: now also C1.1, C2.2, C3.1, C5.1, U4.2 (GND); no longer J1.3 (Pin_3), J2.1 (Pin_1), J5.2 (Pin_2)
- net at J3.1 (Pin_1), PS1.1 (AC/L): now also J2.1 (Pin_1); no longer J2.2 (Pin_2)
- net at J1.2 (Pin_2): now also J2.2 (Pin_2); no longer J4.1 (Pin_1)
- net +3V3: now reaches J6.2 (Pin_2), U3.P1_15 (3V3)
- net +3V3: now also J5.1 (Pin_1), C5.2, U4.1 (Vin)
- net at U3.P1_9 (AIN4/VREFB/EINT/PA04): now also J5.2 (Pin_2), R1.1
- net at U3.P2_10 (PA15/EINT): now also J6.1 (Pin_1), R4.1
- net at U3.P2_4 (PA17/EINT/I2C): now also U4.4 (CLK)
- net at J6.3 (Pin_3), R3.2: now also U3.P2_9 (PA20/EINT/I2SSC); no longer U3.P2_5 (PA19/EINT/I2SD0)
- net at U3.P2_7 (PA18/EINT): now also U4.7 (CS)
- new net: J1.3 (Pin_3), J4.1 (Pin_1)
- new net: U3.P2_5 (PA19/EINT/I2SD0), U4.5 (SDO)
- new net: U3.P2_6 (PA16/EINT/I2C), U4.6 (SDI)
- no-connect marks 21 -> 19
Other:
- moved on the sheet: J6, R3, R4

Commit message: pcb design seems finished
Parts:
- added ACG1, DCG1: TestPoint, TestPoint:TestPoint_THTPad_3.0x3.0mm_Drill1.5mm, symbol Connector:TestPoint
Connections:
- net GND: now also DCG1.1
- net at J1.2 (Pin_2), J2.2 (Pin_2): now also ACG1.1
Changed lines of the file:
@@
 	3250 2100 3250 2050
 Wire Wire Line
-	3250 2050 4700 2050
+	3250 2050 3750 2050
 Wire Wire Line
 	4700 2050 4700 2100
@@
 	4700 2000 4650 2000
 $Comp
-L power:GND #PWR?
+L power:GND #PWR0101
 U 1 1 61CE87CC
 P 7400 3750
-F 0 "#PWR?" H 7400 3500 50  0001 C CNN
+F 0 "#PWR0101" H 7400 3500 50  0001 C CNN
 F 1 "GND" V 7405 3622 50  0000 R CNN
 F 2 "" H 7400 3750 50  0001 C CNN
@@
 	0    -1   -1   0
 $EndComp
+$Comp
+L Connector:TestPoint ACG1
+U 1 1 61D412C6
+P 3750 1300
+F 0 "ACG1" H 3808 1418 50  0000 L CNN
+F 1 "TestPoint" H 3808 1327 50  0000 L CNN
+F 2 "TestPoint:TestPoint_THTPad_3.0x3.0mm_Drill1.5mm" H 3950 1300 50  0001 C CNN
+F 3 "~" H 3950 1300 50  0001 C CNN
+	1    3750 1300
+	1    0    0    -1
+$EndComp
+$Comp
+L Connector:TestPoint DCG1
+U 1 1 61D41B23
+P 4350 1300
+F 0 "DCG1" H 4408 1418 50  0000 L CNN
+F 1 "TestPoint" H 4408 1327 50  0000 L CNN
+F 2 "TestPoint:TestPoint_THTPad_3.0x3.0mm_Drill1.5mm" H 4550 1300 50  0001 C CNN
+F 3 "~" H 4550 1300 50  0001 C CNN
+	1    4350 1300
+	1    0    0    -1
+$EndComp
+$Comp
+L power:GND #PWR0102
+U 1 1 61D41EA8
+P 4350 1300
+F 0 "#PWR0102" H 4350 1050 50  0001 C CNN
+F 1 "GND" H 4355 1127 50  0000 C CNN
+F 2 "" H 4350 1300 50  0001 C CNN
+F 3 "" H 4350 1300 50  0001 C CNN
+	1    4350 1300
+	1    0    0    -1
+$EndComp
+Wire Wire Line
+	3750 1300 3750 2050
+Connection ~ 3750 2050
+Wire Wire Line
+	3750 2050 4700 2050
 $EndSCHEMATC
