File: schematics/cubeSchem/blinky-refrig-mon-cube.kicad_pcb (KiCad board)
At the start: 2 copper layers, 125 x 78 mm, 27 parts, among them J1 VACout, J2 VACin, J3 CTin, J4 CTout, J5 Reed, J6 TripStatus, J7 SMA Ant, U2 ACS712_20, U3 FEATHER_M0_BASIC_PROTO, U4 AMAX31865

Commit message: fixed lora footprint
Parts:
- removed G***: LOGO, dmcginnis427Footprints:blmcLogo2_bs
- removed G***: LOGO, dmcginnis427Footprints:blmcLogo
- removed Lipo1500bs: Lipo1500_bs, dmcginnis427Footprints:Lipo1500_bs
- removed Lipo1500fs: Lipo1500, dmcginnis427Footprints:Lipo1500
- removed U3: FEATHER_M0_BASIC_PROTO, FEATHER_M0_BASIC_PROTO:MODULE_FEATHER_M0_BASIC_PROTO
- added U1: FeatherM0LoRa, dmcginnis427Footprints:FeatherM0LoRa, F.Cu at (188.3, 116.8)
Routing:
- net Net-(R5-Pad1): track 45.6 -> 48.0 mm
- net Net-(J5-Pad2): track 65.7 -> 66.7 mm
